Commit message: update robot param

File: config/robot.urdf.xacro (robot description, xacro)
@@ -17,7 +17,7 @@
   <link name="imu_link"> </link>
   <joint name="imu_joint" type="fixed">
-    <parent link="chassis_link" />
+    <parent link="base_link" />
     <child link="imu_link" />
-    <origin xyz="0 0 0" rpy="0 0 0" />
+    <origin xyz="-1.5 0 0" rpy="3.14158 0 3.14158" />
   </joint>
   <link name="laser_sensor_frame"> </link>
@@ -33,3 +33,9 @@
     <origin xyz="0 0 0" rpy="0 0 0" />
   </joint>
+   <link name="ouster_sensor_center"> </link>
+  <joint name="ouster_joint" type="fixed">
+    <parent link="base_link" />
+    <child link="ouster_sensor_center" />
+    <origin xyz="0 0 1.13" rpy="0 0 0" />
+  </joint>
 </robot>
